Commit message: iiwa14 dual mod

File: iiwa_description/urdf/iiwa.gazebo.xacro (robot description, xacro)
@@ -3,13 +3,25 @@
   <xacro:macro name="iiwa_gazebo" params="robot_name">
      <!-- Enable the Joint Feedback -->
-    <gazebo reference="${robot_name}_joint_7">
+    <gazebo reference="${robot_name}_larm_joint_7">
+      <provideFeedback>true</provideFeedback>
+    </gazebo>
+     <!-- Enable the Joint Feedback -->
+    <gazebo reference="${robot_name}_rarm_joint_7">
       <provideFeedback>true</provideFeedback>
     </gazebo>
     <!-- The ft_sensor plugin -->
     <gazebo>
-      <plugin name="ft_sensor" filename="libgazebo_ros_ft_sensor.so">
+      <plugin name="larm_ft_sensor" filename="libgazebo_ros_ft_sensor.so">
         <updateRate>50.0</updateRate>
         <topicName>/${robot_name}/state/CartesianWrench</topicName>
-        <jointName>${robot_name}_joint_7</jointName>
+        <jointName>${robot_name}_larm_joint_7</jointName>
+      </plugin>
+    </gazebo>
+    <!-- The ft_sensor plugin -->
+    <gazebo>
+      <plugin name="rarm_ft_sensor" filename="libgazebo_ros_ft_sensor.so">
+        <updateRate>50.0</updateRate>
+        <topicName>/${robot_name}/state/CartesianWrench</topicName>
+        <jointName>${robot_name}_rarm_joint_7</jointName>
       </plugin>
     </gazebo>
@@ -21,5 +33,5 @@
     </gazebo>
     <!-- Link0 -->
-    <gazebo reference="${robot_name}_link_0">
+    <gazebo reference="${robot_name}_larm_link_0">
       <material>Gazebo/Grey</material>
       <mu1>0.2</mu1>
@@ -27,5 +39,5 @@
     </gazebo>
     <!-- Link1 -->
-    <gazebo reference="${robot_name}_link_1">
+    <gazebo reference="${robot_name}_larm_link_1">
       <material>Gazebo/Orange</material>
       <mu1>0.2</mu1>
@@ -33,5 +45,5 @@
     </gazebo>
     <!-- Link2 -->
-    <gazebo reference="${robot_name}_link_2">
+    <gazebo reference="${robot_name}_larm_link_2">
       <material>Gazebo/Orange</material>
       <mu1>0.2</mu1>
@@ -39,5 +51,5 @@
     </gazebo>
     <!-- Link3 -->
-    <gazebo reference="${robot_name}_link_3">
+    <gazebo reference="${robot_name}_larm_link_3">
       <material>Gazebo/Orange</material>
       <mu1>0.2</mu1>
@@ -45,5 +57,5 @@
     </gazebo>
     <!-- Link4 -->
-    <gazebo reference="${robot_name}_link_4">
+    <gazebo reference="${robot_name}_larm_link_4">
       <material>Gazebo/Orange</material>
       <mu1>0.2</mu1>
@@ -51,5 +63,5 @@
     </gazebo>
     <!-- Link5 -->
-    <gazebo reference="${robot_name}_link_5">
+    <gazebo reference="${robot_name}_larm_link_5">
       <material>Gazebo/Orange</material>
       <mu1>0.2</mu1>
@@ -57,5 +69,5 @@
     </gazebo>
     <!-- Link6 -->
-    <gazebo reference="${robot_name}_link_6">
+    <gazebo reference="${robot_name}_larm_link_6">
       <material>Gazebo/Orange</material>
       <mu1>0.2</mu1>
@@ -63,5 +75,53 @@
     </gazebo>
     <!-- Link7 -->
-    <gazebo reference="${robot_name}_link_7">
+    <gazebo reference="${robot_name}_larm_link_7">
+      <material>Gazebo/Grey</material>
+      <mu1>0.2</mu1>
+      <mu2>0.2</mu2>
+    </gazebo>
+    <!-- Link0 -->
+    <gazebo reference="${robot_name}_rarm_link_0">
+      <material>Gazebo/Grey</material>
+      <mu1>0.2</mu1>
+      <mu2>0.2</mu2>
+    </gazebo>
+    <!-- Link1 -->
+    <gazebo reference="${robot_name}_rarm_link_1">
+      <material>Gazebo/Orange</material>
+      <mu1>0.2</mu1>
+      <mu2>0.2</mu2>
+    </gazebo>
+    <!-- Link2 -->
+    <gazebo reference="${robot_name}_rarm_link_2">
+      <material>Gazebo/Orange</material>
+      <mu1>0.2</mu1>
+      <mu2>0.2</mu2>
+    </gazebo>
+    <!-- Link3 -->
+    <gazebo reference="${robot_name}_rarm_link_3">
+      <material>Gazebo/Orange</material>
+      <mu1>0.2</mu1>
+      <mu2>0.2</mu2>
+    </gazebo>
+    <!-- Link4 -->
+    <gazebo reference="${robot_name}_rarm_link_4">
+      <material>Gazebo/Orange</material>
+      <mu1>0.2</mu1>
+      <mu2>0.2</mu2>
+    </gazebo>
+    <!-- Link5 -->
+    <gazebo reference="${robot_name}_rarm_link_5">
+      <material>Gazebo/Orange</material>
+      <mu1>0.2</mu1>
+      <mu2>0.2</mu2>
+    </gazebo>
+    <!-- Link6 -->
+    <gazebo reference="${robot_name}_rarm_link_6">
+      <material>Gazebo/Orange</material>
+      <mu1>0.2</mu1>
+      <mu2>0.2</mu2>
+    </gazebo>
+    <!-- Link7 -->
+    <gazebo reference="${robot_name}_rarm_link_7">
       <material>Gazebo/Grey</material>
       <mu1>0.2</mu1>

File: iiwa_description/urdf/iiwa.transmission.xacro (robot description, xacro)
@@ -2,77 +2,154 @@
 <robot xmlns:xacro="http://www.ros.org/wiki/xacro">
   <xacro:macro name="iiwa_transmission" params="hardware_interface">
-    <transmission name="${robot_name}_tran_1">
+    <transmission name="${robot_name}_larm_tran_1">
       <robotNamespace>/${robot_name}</robotNamespace>
       <type>transmission_interface/SimpleTransmission</type>
-      <joint name="${robot_name}_joint_1">
+      <joint name="${robot_name}_larm_joint_1">
         <hardwareInterface>hardware_interface/${hardware_interface}</hardwareInterface>
       </joint>
-      <actuator name="${robot_name}_motor_1">
+      <actuator name="${robot_name}_larm_motor_1">
         <hardwareInterface>hardware_interface/${hardware_interface}</hardwareInterface>
         <mechanicalReduction>1</mechanicalReduction>
       </actuator>
     </transmission>
-    <transmission name="${robot_name}_tran_2">
+    <transmission name="${robot_name}_larm_tran_2">
       <robotNamespace>/${robot_name}</robotNamespace>
       <type>transmission_interface/SimpleTransmission</type>
-      <joint name="${robot_name}_joint_2">
+      <joint name="${robot_name}_larm_joint_2">
         <hardwareInterface>hardware_interface/${hardware_interface}</hardwareInterface>
       </joint>
-      <actuator name="${robot_name}_motor_2">
+      <actuator name="${robot_name}_larm_motor_2">
         <hardwareInterface>hardware_interface/${hardware_interface}</hardwareInterface>
         <mechanicalReduction>1</mechanicalReduction>
       </actuator>
     </transmission>
-    <transmission name="${robot_name}_tran_3">
+    <transmission name="${robot_name}_larm_tran_3">
       <robotNamespace>/${robot_name}</robotNamespace>
       <type>transmission_interface/SimpleTransmission</type>
-      <joint name="${robot_name}_joint_3">
+      <joint name="${robot_name}_larm_joint_3">
         <hardwareInterface>hardware_interface/${hardware_interface}</hardwareInterface>
       </joint>
-      <actuator name="${robot_name}_motor_3">
+      <actuator name="${robot_name}_larm_motor_3">
         <hardwareInterface>hardware_interface/${hardware_interface}</hardwareInterface>
         <mechanicalReduction>1</mechanicalReduction>
       </actuator>
     </transmission>
-    <transmission name="${robot_name}_tran_4">
+    <transmission name="${robot_name}_larm_tran_4">
       <robotNamespace>/${robot_name}</robotNamespace>
       <type>transmission_interface/SimpleTransmission</type>
-      <joint name="${robot_name}_joint_4">
+      <joint name="${robot_name}_larm_joint_4">
         <hardwareInterface>hardware_interface/${hardware_interface}</hardwareInterface>
       </joint>
-      <actuator name="${robot_name}_motor_4">
+      <actuator name="${robot_name}_larm_motor_4">
         <hardwareInterface>hardware_interface/${hardware_interface}</hardwareInterface>
         <mechanicalReduction>1</mechanicalReduction>
       </actuator>
     </transmission>
-    <transmission name="${robot_name}_tran_5">
+    <transmission name="${robot_name}_larm_tran_5">
       <robotNamespace>/${robot_name}</robotNamespace>
       <type>transmission_interface/SimpleTransmission</type>
-      <joint name="${robot_name}_joint_5">
+      <joint name="${robot_name}_larm_joint_5">
         <hardwareInterface>hardware_interface/${hardware_interface}</hardwareInterface>
       </joint>
-      <actuator name="${robot_name}_motor_5">
+      <actuator name="${robot_name}_larm_motor_5">
         <hardwareInterface>hardware_interface/${hardware_interface}</hardwareInterface>
         <mechanicalReduction>1</mechanicalReduction>
       </actuator>
     </transmission>
-    <transmission name="${robot_name}_tran_6">
+    <transmission name="${robot_name}_larm_tran_6">
       <robotNamespace>/${robot_name}</robotNamespace>
       <type>transmission_interface/SimpleTransmission</type>
-      <joint name="${robot_name}_joint_6">
+      <joint name="${robot_name}_larm_joint_6">
         <hardwareInterface>hardware_interface/${hardware_interface}</hardwareInterface>
       </joint>
-      <actuator name="${robot_name}_motor_6">
+      <actuator name="${robot_name}_larm_motor_6">
         <hardwareInterface>hardware_interface/${hardware_interface}</hardwareInterface>
         <mechanicalReduction>1</mechanicalReduction>
       </actuator>
     </transmission>
-    <transmission name="${robot_name}_tran_7">
+    <transmission name="${robot_name}_larm_tran_7">
       <robotNamespace>/${robot_name}</robotNamespace>
       <type>transmission_interface/SimpleTransmission</type>
-      <joint name="${robot_name}_joint_7">
+      <joint name="${robot_name}_larm_joint_7">
         <hardwareInterface>hardware_interface/${hardware_interface}</hardwareInterface>
       </joint>
-      <actuator name="${robot_name}_motor_7">
+      <actuator name="${robot_name}_larm_motor_7">
+        <hardwareInterface>hardware_interface/${hardware_interface}</hardwareInterface>
+        <mechanicalReduction>1</mechanicalReduction>
+      </actuator>
+    </transmission>
+    <transmission name="${robot_name}_rarm_tran_1">
+      <robotNamespace>/${robot_name}</robotNamespace>
+      <type>transmission_interface/SimpleTransmission</type>
+      <joint name="${robot_name}_rarm_joint_1">
+        <hardwareInterface>hardware_interface/${hardware_interface}</hardwareInterface>
+      </joint>
+      <actuator name="${robot_name}_rarm_motor_1">
+        <hardwareInterface>hardware_interface/${hardware_interface}</hardwareInterface>
+        <mechanicalReduction>1</mechanicalReduction>
+      </actuator>
+    </transmission>
+    <transmission name="${robot_name}_rarm_tran_2">
+      <robotNamespace>/${robot_name}</robotNamespace>
+      <type>transmission_interface/SimpleTransmission</type>
+      <joint name="${robot_name}_rarm_joint_2">
+        <hardwareInterface>hardware_interface/${hardware_interface}</hardwareInterface>
+      </joint>
+      <actuator name="${robot_name}_rarm_motor_2">
+        <hardwareInterface>hardware_interface/${hardware_interface}</hardwareInterface>
+        <mechanicalReduction>1</mechanicalReduction>
+      </actuator>
+    </transmission>
+    <transmission name="${robot_name}_rarm_tran_3">
+      <robotNamespace>/${robot_name}</robotNamespace>
+      <type>transmission_interface/SimpleTransmission</type>
+      <joint name="${robot_name}_rarm_joint_3">
+        <hardwareInterface>hardware_interface/${hardware_interface}</hardwareInterface>
+      </joint>
+      <actuator name="${robot_name}_rarm_motor_3">
+        <hardwareInterface>hardware_interface/${hardware_interface}</hardwareInterface>
+        <mechanicalReduction>1</mechanicalReduction>
+      </actuator>
+    </transmission>
+    <transmission name="${robot_name}_rarm_tran_4">
+      <robotNamespace>/${robot_name}</robotNamespace>
+      <type>transmission_interface/SimpleTransmission</type>
+      <joint name="${robot_name}_rarm_joint_4">
+        <hardwareInterface>hardware_interface/${hardware_interface}</hardwareInterface>
+      </joint>
+      <actuator name="${robot_name}_rarm_motor_4">
+        <hardwareInterface>hardware_interface/${hardware_interface}</hardwareInterface>
+        <mechanicalReduction>1</mechanicalReduction>
+      </actuator>
+    </transmission>
+    <transmission name="${robot_name}_rarm_tran_5">
+      <robotNamespace>/${robot_name}</robotNamespace>
+      <type>transmission_interface/SimpleTransmission</type>
+      <joint name="${robot_name}_rarm_joint_5">
+        <hardwareInterface>hardware_interface/${hardware_interface}</hardwareInterface>
+      </joint>
+      <actuator name="${robot_name}_rarm_motor_5">
+        <hardwareInterface>hardware_interface/${hardware_interface}</hardwareInterface>
+        <mechanicalReduction>1</mechanicalReduction>
+      </actuator>
+    </transmission>
+    <transmission name="${robot_name}_rarm_tran_6">
+      <robotNamespace>/${robot_name}</robotNamespace>
+      <type>transmission_interface/SimpleTransmission</type>
+      <joint name="${robot_name}_rarm_joint_6">
+        <hardwareInterface>hardware_interface/${hardware_interface}</hardwareInterface>
+      </joint>
+      <actuator name="${robot_name}_rarm_motor_6">
+        <hardwareInterface>hardware_interface/${hardware_interface}</hardwareInterface>
+        <mechanicalReduction>1</mechanicalReduction>
+      </actuator>
+    </transmission>
+    <transmission name="${robot_name}_rarm_tran_7">
+      <robotNamespace>/${robot_name}</robotNamespace>
+      <type>transmission_interface/SimpleTransmission</type>
+      <joint name="${robot_name}_rarm_joint_7">
+        <hardwareInterface>hardware_interface/${hardware_interface}</hardwareInterface>
+      </joint>
+      <actuator name="${robot_name}_rarm_motor_7">
         <hardwareInterface>hardware_interface/${hardware_interface}</hardwareInterface>
         <mechanicalReduction>1</mechanicalReduction>
