Commit message: add camera

File: iiwa_description/urdf/iiwad.gazebo.xacro (robot description, xacro)
@@ -9,4 +9,70 @@
     <gazebo reference="${robot_name}_rarm_joint_7">
       <provideFeedback>true</provideFeedback>
+    </gazebo>
+    <gazebo reference="${robot_name}_larm_link_ee">
+      <material>Gazebo/Grey</material>
+      <mu1>0.2</mu1>
+      <mu2>0.2</mu2>
+    </gazebo>
+    <gazebo reference="${robot_name}_rarm_link_ee">
+      <material>Gazebo/Grey</material>
+      <mu1>0.2</mu1>
+      <mu2>0.2</mu2>
+    </gazebo>
+    <gazebo reference="${robot_name}_torso_link">
+      <sensor type="multicamera" name="stereo_camera">
+	<update_rate>30.0</update_rate>
+	<camera name="left">
+	  <pose>0.424264 0.03 1.6 0 ${radians(45)} 0</pose>
+          <horizontal_fov>1.3962634</horizontal_fov>
+          <image>
+            <width>800</width>
+            <height>800</height>
+            <format>R8G8B8</format>
+          </image>
+          <clip>
+            <near>0.02</near>
+            <far>300</far>
+          </clip>
+          <noise>
+            <type>gaussian</type>
+            <mean>0.0</mean>
+            <stddev>0.007</stddev>
+          </noise>
+	</camera>
+	<camera name="right">
+          <pose>0 -0.03 1.6 0 ${radians(45)} 0</pose>
+          <horizontal_fov>1.3962634</horizontal_fov>
+          <image>
+            <width>800</width>
+            <height>800</height>
+            <format>R8G8B8</format>
+          </image>
+          <clip>
+            <near>0.02</near>
+            <far>300</far>
+          </clip>
+          <noise>
+            <type>gaussian</type>
+            <mean>0.0</mean>
+            <stddev>0.007</stddev>
+          </noise>
+	</camera>
+	<plugin name="stereo_camera_controller" filename="libgazebo_ros_multicamera.so">
+          <alwaysOn>true</alwaysOn>
+          <updateRate>0.0</updateRate>
+          <cameraName>${robot_name}/camera</cameraName>
+          <imageTopicName>image_raw</imageTopicName>
+          <cameraInfoTopicName>camera_info</cameraInfoTopicName>
+          <frameName>left_camera_optical_frame</frameName>
+          <!--<rightFrameName>right_camera_optical_frame</rightFrameName>-->
+          <hackBaseline>0.07</hackBaseline>
+          <distortionK1>0.0</distortionK1>
+          <distortionK2>0.0</distortionK2>
+          <distortionK3>0.0</distortionK3>
+          <distortionT1>0.0</distortionT1>
+          <distortionT2>0.0</distortionT2>
+	</plugin>
+      </sensor>
     </gazebo>
     <!-- use hrpsys_gazebo_plugin instead of these -->
